File: PCB_design/turner_pcb/turner_pcb/turner_pcb.kicad_pcb (KiCad board)
At the start: 2 copper layers, 17.8 x 43.2 mm, 6 parts, among them P1 Digital, P2 Analog, P3 CONN_01X01, P4 CONN_01X01, P5 CONN_01X01, P6 CONN_01X01

Commit message: First version of working firmware.
Other:
- board size 17.8 x 43.2 mm -> 79.1 x 90 mm
Changed lines of the file:
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@@
-(kicad_pcb (version 4) (host pcbnew 4.0.4+e1-6308~48~ubuntu14.04.1-stable)
+(kicad_pcb (version 20171130) (host pcbnew "(5.1.5)-3")
   (general
-    (links 2)
-    (no_connects 2)
-    (area 138.125999 67.386999 156.006001 110.667001)
     (thickness 1.6)
-    (drawings 20)
+    (drawings 24)
     (tracks 0)
     (zones 0)
@@
     (zone_45_only no)
     (trace_min 0.2)
-    (segment_width 0.15)
-    (edge_width 0.1)
     (via_size 0.6)
     (via_drill 0.4)
@@
     (uvia_min_size 0.2)
     (uvia_min_drill 0.1)
+    (edge_width 0.1)
+    (segment_width 0.15)
     (pcb_text_width 0.3)
     (pcb_text_size 1.5 1.5)
@@
     (pad_to_mask_clearance 0)
     (aux_axis_origin 138.176 110.617)
-    (visible_elements FFFFFF7F)
+    (visible_elements 7FFFFFFF)
     (pcbplotparams
       (layerselection 0x00030_80000001)
       (usegerberextensions false)
+      (usegerberattributes false)
+      (usegerberadvancedattributes false)
+      (creategerberjobfile false)
       (excludeedgelayer true)
       (linewidth 0.100000)
@@
       (hpglpennumber 1)
       (hpglpenspeed 20)
-      (hpglpendiameter 15)
-      (hpglpenoverlay 2)
+      (hpglpendiameter 15.000000)
       (psnegative false)
       (psa4output false)
@@
       (net 32 "/12(MISO)"))
     (model ${KIPRJMOD}/Socket_Arduino_Nano.3dshapes/Socket_header_Arduino_1x15.wrl
-      (at (xyz 0.7 0 0))
+      (offset (xyz 17.77999973297119 0 0))
       (scale (xyz 1 1 1))
       (rotate (xyz 0 0 180))
@@
       (net 25 "/13(SCK)"))
     (model ${KIPRJMOD}/Socket_Arduino_Nano.3dshapes/Socket_header_Arduino_1x15.wrl
-      (at (xyz 0.7 0 0))
+      (offset (xyz 17.77999973297119 0 0))
       (scale (xyz 1 1 1))
       (rotate (xyz 0 0 180))
@@
       (net 29 "Net-(P6-Pad1)"))
   )
+  (gr_line (start 116.205 40.2082) (end 113.4872 130.2004) (layer Edge.Cuts) (width 0.1))
+  (gr_line (start 192.6082 40.2082) (end 116.205 40.2082) (layer Edge.Cuts) (width 0.1))
+  (gr_line (start 192.2272 130.2004) (end 192.6082 40.2082) (layer Edge.Cuts) (width 0.1))
+  (gr_line (start 113.4872 130.2004) (end 192.2272 130.2004) (layer Edge.Cuts) (width 0.1))
   (gr_text 1 (at 141.732 71.247) (layer F.SilkS)
     (effects (font (size 1 1) (thickness 0.15)))
